File: pcb/stm8_card.sch (KiCad schematic (older format))
At the start: 20 parts

Commit message: pcb finished first schematic revision
Parts:
- added C?: 1uf, symbol Device:C_Small
- J?: value Conn_01x08 -> DEBUG HEADER
- SW? (x3): value SW_Push -> TL59AF100Q; digikey TL59AF100Q -> EG4378CT-ND
- SW?: value SW_Push -> TL3302AF260QG; digikey TL59AF100Q -> EG4584CT-ND
Connections:
- net labels added: RX, SWIM, TX
- wire segments 81 -> 94
Changed lines of the file:
@@
 P 3950 4050
 F 0 "SW?" H 3950 4335 50  0000 C CNN
-F 1 "SW_Push" H 3950 4334 50  0001 C CNN
+F 1 "TL59AF100Q" H 3950 4334 50  0001 C CNN
 F 2 "" H 3950 4250 50  0001 C CNN
 F 3 "~" H 3950 4250 50  0001 C CNN
-F 4 "TL59AF100Q" H 3950 4244 50  0000 C CNN "digikey"
+F 4 "EG4378CT-ND" H 3950 4244 50  0000 C CNN "digikey"
 	1    3950 4050
 	1    0    0    -1
@@
 P 3950 4950
 F 0 "SW?" H 3950 5235 50  0000 C CNN
-F 1 "SW_Push" H 3950 5234 50  0001 C CNN
+F 1 "TL59AF100Q" H 3950 5234 50  0001 C CNN
 F 2 "" H 3950 5150 50  0001 C CNN
 F 3 "~" H 3950 5150 50  0001 C CNN
-F 4 "TL59AF100Q" H 3950 5144 50  0000 C CNN "digikey"
+F 4 "EG4378CT-ND" H 3950 5144 50  0000 C CNN "digikey"
 	1    3950 4950
 	1    0    0    -1
@@
 P 3950 4500
 F 0 "SW?" H 3950 4785 50  0000 C CNN
-F 1 "SW_Push" H 3950 4784 50  0001 C CNN
+F 1 "TL59AF100Q" H 3950 4784 50  0001 C CNN
 F 2 "" H 3950 4700 50  0001 C CNN
 F 3 "~" H 3950 4700 50  0001 C CNN
-F 4 "TL59AF100Q" H 3950 4694 50  0000 C CNN "digikey"
+F 4 "EG4378CT-ND" H 3950 4694 50  0000 C CNN "digikey"
 	1    3950 4500
 	1    0    0    -1
@@
 L power:GND #PWR?
 U 1 1 6081EBFF
-P 1300 4600
-F 0 "#PWR?" H 1300 4350 50  0001 C CNN
-F 1 "GND" H 1305 4427 50  0000 C CNN
-F 2 "" H 1300 4600 50  0001 C CNN
-F 3 "" H 1300 4600 50  0001 C CNN
-	1    1300 4600
+P 4700 2100
+F 0 "#PWR?" H 4700 1850 50  0001 C CNN
+F 1 "GND" H 4705 1927 50  0000 C CNN
+F 2 "" H 4700 2100 50  0001 C CNN
+F 3 "" H 4700 2100 50  0001 C CNN
+	1    4700 2100
 	1    0    0    -1
 $EndComp
@@
 L power:GND #PWR?
 U 1 1 6082B314
-P 8100 3850
-F 0 "#PWR?" H 8100 3600 50  0001 C CNN
-F 1 "GND" H 8105 3677 50  0000 C CNN
-F 2 "" H 8100 3850 50  0001 C CNN
-F 3 "" H 8100 3850 50  0001 C CNN
-	1    8100 3850
-	1    0    0    -1
-$EndComp
-Wire Wire Line
-	8100 3700 8100 3850
+P 8100 3750
+F 0 "#PWR?" H 8100 3500 50  0001 C CNN
+F 1 "GND" H 8105 3577 50  0000 C CNN
+F 2 "" H 8100 3750 50  0001 C CNN
+F 3 "" H 8100 3750 50  0001 C CNN
+	1    8100 3750
+	1    0    0    -1
+$EndComp
 $Comp
 L Device:C_Small C?
@@
 U 1 1 60827F4F
 P 6300 4650
-F 0 "SW?" H 6300 4935 50  0000 C CNN
-F 1 "SW_Push" H 6300 4934 50  0001 C CNN
+F 0 "SW?" H 6300 4950 50  0000 C CNN
+F 1 "TL3302AF260QG" H 6300 4934 50  0001 C CNN
 F 2 "" H 6300 4850 50  0001 C CNN
 F 3 "~" H 6300 4850 50  0001 C CNN
-F 4 "TL59AF100Q" H 6300 4844 50  0000 C CNN "digikey"
+F 4 "EG4584CT-ND" H 6300 4844 50  0000 C CNN "digikey"
 	1    6300 4650
 	1    0    0    -1
@@
 Text GLabel 6600 4650 2    50   Input ~ 0
 NRST
-Text GLabel 7050 3000 0    50   Input ~ 0
+Text GLabel 7250 3000 0    50   Input ~ 0
 NRST
 Text GLabel 3150 2800 2    50   Input ~ 0
 NRST
 Wire Wire Line
-	7050 3000 7400 3000
+	7250 3000 7400 3000
 Text GLabel 2450 1300 0    50   Input ~ 0
 3v3
@@
 P 5250 1650
 F 0 "J?" H 5330 1642 50  0000 L CNN
-F 1 "Conn_01x08" H 5330 1551 50  0000 L CNN
+F 1 "DEBUG HEADER" H 5330 1551 50  0000 L CNN
 F 2 "" H 5250 1650 50  0001 C CNN
 F 3 "~" H 5250 1650 50  0001 C CNN
@@
 	1    0    0    -1
 $EndComp
+Text GLabel 4750 1350 0    50   Input ~ 0
+3v3
+Wire Wire Line
+	5050 1350 4750 1350
+Wire Wire Line
+	5050 2050 4700 2050
+Wire Wire Line
+	4700 2050 4700 2100
+Text GLabel 4750 1450 0    50   Input ~ 0
+TX
+Text GLabel 7250 2700 0    50   Input ~ 0
+TX
+Text GLabel 4750 1550 0    50   Input ~ 0
+RX
+Text GLabel 7250 2800 0    50   Input ~ 0
+RX
+Wire Wire Line
+	4750 1450 5050 1450
+Wire Wire Line
+	4750 1550 5050 1550
+Text GLabel 4750 1650 0    50   Input ~ 0
+SWIM
+Wire Wire Line
+	4750 1650 5050 1650
+Text GLabel 4750 1750 0    50   Input ~ 0
+NRST
+Wire Wire Line
+	4750 1750 5050 1750
+Text GLabel 9100 2750 2    50   Input ~ 0
+SWIM
+Wire Wire Line
+	9100 2750 8850 2750
+Wire Wire Line
+	7250 2700 7400 2700
+Wire Wire Line
+	7250 2800 7400 2800
+$Comp
+L Device:C_Small C?
+U 1 1 608B409C
+P 7100 3550
+F 0 "C?" H 7192 3596 50  0000 L CNN
+F 1 "1uf" H 7192 3505 50  0000 L CNN
+F 2 "" H 7100 3550 50  0001 C CNN
+F 3 "~" H 7100 3550 50  0001 C CNN
+	1    7100 3550
+	1    0    0    -1
+$EndComp
+Wire Wire Line
+	7400 3400 7100 3400
+$Comp
+L power:GND #PWR?
+U 1 1 608B7854
+P 7100 3750
+F 0 "#PWR?" H 7100 3500 50  0001 C CNN
+F 1 "GND" H 7105 3577 50  0000 C CNN
+F 2 "" H 7100 3750 50  0001 C CNN
+F 3 "" H 7100 3750 50  0001 C CNN
+	1    7100 3750
+	1    0    0    -1
+$EndComp
+Wire Wire Line
+	7100 3750 7100 3650
+Wire Wire Line
+	7100 3450 7100 3400
+Wire Wire Line
+	8100 3750 8100 3700
 $EndSCHEMATC
