File: pcb/stm8_card.sch (KiCad schematic (older format))
At the start: 31 parts, among them J1 DEBUG HEADER, SW1 TL59AF100Q, SW2 TL59AF100Q, SW3 TL59AF100Q, SW4 TL3302AF260QG, U1 ER-OLED0.91-7, U2 STM8S103F3

Commit message: annotated components
Parts:
- gave numbers to parts that had none: 6
Other:
- moved on the sheet: C10, D1, R7
Changed lines of the file:
@@
 Wire Wire Line
 	4800 4500 4800 4950
-Text GLabel 5200 6500 0    50   Input ~ 0
+Text GLabel 1650 3900 0    50   Input ~ 0
 3v3
 Text GLabel 3450 3950 0    50   Input ~ 0
@@
 L stm8_card-rescue:GND-power #PWR01
 U 1 1 60827C7E
-P 6200 6650
-F 0 "#PWR01" H 6200 6400 50  0001 C CNN
-F 1 "GND" H 6205 6477 50  0000 C CNN
-F 2 "" H 6200 6650 50  0001 C CNN
-F 3 "" H 6200 6650 50  0001 C CNN
-	1    6200 6650
+P 2650 4050
+F 0 "#PWR01" H 2650 3800 50  0001 C CNN
+F 1 "GND" H 2655 3877 50  0000 C CNN
+F 2 "" H 2650 4050 50  0001 C CNN
+F 3 "" H 2650 4050 50  0001 C CNN
+	1    2650 4050
 	1    0    0    -1
 $EndComp
@@
 L stm8_card-rescue:PWR_FLAG-power #FLG01
 U 1 1 6084AA5A
-P 5250 6650
-F 0 "#FLG01" H 5250 6725 50  0001 C CNN
-F 1 "PWR_FLAG" V 5250 6777 50  0000 L CNN
-F 2 "" H 5250 6650 50  0001 C CNN
-F 3 "~" H 5250 6650 50  0001 C CNN
-	1    5250 6650
+P 1700 4050
+F 0 "#FLG01" H 1700 4125 50  0001 C CNN
+F 1 "PWR_FLAG" V 1700 4177 50  0000 L CNN
+F 2 "" H 1700 4050 50  0001 C CNN
+F 3 "~" H 1700 4050 50  0001 C CNN
+	1    1700 4050
 	0    -1   -1   0
 $EndComp
@@
 L stm8_card-rescue:PWR_FLAG-power #FLG02
 U 1 1 6084B498
-P 5250 7050
-F 0 "#FLG02" H 5250 7125 50  0001 C CNN
-F 1 "PWR_FLAG" V 5250 7177 50  0000 L CNN
-F 2 "" H 5250 7050 50  0001 C CNN
-F 3 "~" H 5250 7050 50  0001 C CNN
-	1    5250 7050
+P 1700 4450
+F 0 "#FLG02" H 1700 4525 50  0001 C CNN
+F 1 "PWR_FLAG" V 1700 4577 50  0000 L CNN
+F 2 "" H 1700 4450 50  0001 C CNN
+F 3 "~" H 1700 4450 50  0001 C CNN
+	1    1700 4450
 	0    -1   -1   0
 $EndComp
 Wire Wire Line
-	5200 6500 5250 6500
-Wire Wire Line
-	5250 6500 5250 6650
-Wire Wire Line
-	5250 6700 5250 6650
-Connection ~ 5250 6650
-Wire Wire Line
-	5250 7000 5250 7050
-Connection ~ 5250 7050
+	1650 3900 1700 3900
+Wire Wire Line
+	1700 3900 1700 4050
+Wire Wire Line
+	1700 4100 1700 4050
+Connection ~ 1700 4050
+Wire Wire Line
+	1700 4400 1700 4450
+Connection ~ 1700 4450
 Wire Wire Line
 	2050 1300 2050 1400
@@
 L stm8_card-rescue:R-Device R7
 U 1 1 6087FF9F
-P 6000 6500
-F 0 "R7" V 5900 6500 50  0000 C CNN
-F 1 "4.7k" V 6000 6500 50  0000 C CNN
-F 2 "Resistor_SMD:R_0805_2012Metric_Pad1.20x1.40mm_HandSolder" V 5930 6500 50  0001 C CNN
-F 3 "~" H 6000 6500 50  0001 C CNN
-	1    6000 6500
+P 2450 3900
+F 0 "R7" V 2350 3900 50  0000 C CNN
+F 1 "4.7k" V 2450 3900 50  0000 C CNN
+F 2 "Resistor_SMD:R_0805_2012Metric_Pad1.20x1.40mm_HandSolder" V 2380 3900 50  0001 C CNN
+F 3 "~" H 2450 3900 50  0001 C CNN
+	1    2450 3900
 	0    -1   -1   0
 $EndComp
@@
 L stm8_card-rescue:LED-Device D1
 U 1 1 6088C1B4
-P 5650 6500
-F 0 "D1" H 5643 6245 50  0000 C CNN
-F 1 "LED" H 5643 6336 50  0000 C CNN
-F 2 "stm8_card:LED_0805_2012Metric_Pad1.15x1.40mm_HandSolder" H 5650 6500 50  0001 C CNN
-F 3 "~" H 5650 6500 50  0001 C CNN
-F 4 "404-1316-1-ND" H 5650 6500 50  0001 C CNN "digikey"
-	1    5650 6500
+P 2100 3900
+F 0 "D1" H 2093 3645 50  0000 C CNN
+F 1 "LED" H 2093 3736 50  0000 C CNN
+F 2 "stm8_card:LED_0805_2012Metric_Pad1.15x1.40mm_HandSolder" H 2100 3900 50  0001 C CNN
+F 3 "~" H 2100 3900 50  0001 C CNN
+F 4 "404-1316-1-ND" H 2100 3900 50  0001 C CNN "digikey"
+	1    2100 3900
 	-1   0    0    1
 $EndComp
 Wire Wire Line
-	5250 6500 5500 6500
-Connection ~ 5250 6500
-Wire Wire Line
-	5800 6500 5850 6500
-Wire Wire Line
-	6200 6500 6200 6650
-Wire Wire Line
-	6150 6500 6200 6500
-$Comp
-L stm8_card-rescue:GND-power #PWR?
+	1700 3900 1950 3900
+Connection ~ 1700 3900
+Wire Wire Line
+	2250 3900 2300 3900
+Wire Wire Line
+	2650 3900 2650 4050
+Wire Wire Line
+	2600 3900 2650 3900
+$Comp
+L stm8_card-rescue:GND-power #PWR016
 U 1 1 608BFC4F
-P 5250 7250
-F 0 "#PWR?" H 5250 7000 50  0001 C CNN
-F 1 "GND" H 5255 7077 50  0000 C CNN
-F 2 "" H 5250 7250 50  0001 C CNN
-F 3 "" H 5250 7250 50  0001 C CNN
-	1    5250 7250
-	1    0    0    -1
-$EndComp
-Wire Wire Line
-	5250 7050 5250 7250
+P 1700 4650
+F 0 "#PWR016" H 1700 4400 50  0001 C CNN
+F 1 "GND" H 1705 4477 50  0000 C CNN
+F 2 "" H 1700 4650 50  0001 C CNN
+F 3 "" H 1700 4650 50  0001 C CNN
+	1    1700 4650
+	1    0    0    -1
+$EndComp
+Wire Wire Line
+	1700 4450 1700 4650
 $Comp
 L Device:C C10
 U 1 1 60AC16C5
-P 5250 6850
-F 0 "C10" H 5365 6941 50  0000 L CNN
-F 1 "330mF" H 5365 6850 50  0000 L CNN
-F 2 "" H 5288 6700 50  0001 C CNN
-F 3 "~" H 5250 6850 50  0001 C CNN
-F 4 "604-1160-2-ND" H 5365 6759 50  0000 L CNN "digikey"
-	1    5250 6850
-	1    0    0    -1
-$EndComp
-$Comp
-L Connector:USB_C_Receptacle_USB2.0 J?
+P 1700 4250
+F 0 "C10" H 1815 4341 50  0000 L CNN
+F 1 "330mF" H 1815 4250 50  0000 L CNN
+F 2 "" H 1738 4100 50  0001 C CNN
+F 3 "~" H 1700 4250 50  0001 C CNN
+F 4 "604-1160-2-ND" H 1815 4159 50  0000 L CNN "digikey"
+	1    1700 4250
+	1    0    0    -1
+$EndComp
+$Comp
+L Connector:USB_C_Receptacle_USB2.0 J2
 U 1 1 60AD1E79
 P 1200 6450
-F 0 "J?" H 1307 7407 50  0000 C CNN
+F 0 "J2" H 1307 7407 50  0000 C CNN
 F 1 "USB_C_Receptacle_USB2.0" H 1307 7316 50  0000 C CNN
 F 2 "" H 1350 6450 50  0001 C CNN
@@
 $EndComp
 $Comp
-L Regulator_Linear:MIC5205-3.3YM5 U?
+L Regulator_Linear:MIC5205-3.3YM5 U3
 U 1 1 60AFC40A
 P 2900 6550
-F 0 "U?" H 2900 6983 50  0000 C CNN
+F 0 "U3" H 2900 6983 50  0000 C CNN
 F 1 "MIC5253-3.3YC5" H 2900 6892 50  0000 C CNN
 F 2 "Package_TO_SOT_SMD:SOT-23-5" H 2900 6875 50  0001 C CNN
@@
 Connection ~ 2300 6450
 $Comp
-L stm8_card-rescue:GND-power #PWR?
+L stm8_card-rescue:GND-power #PWR013
 U 1 1 60B05530
 P 2900 7000
-F 0 "#PWR?" H 2900 6750 50  0001 C CNN
+F 0 "#PWR013" H 2900 6750 50  0001 C CNN
 F 1 "GND" H 2905 6827 50  0000 C CNN
 F 2 "" H 2900 7000 50  0001 C CNN
@@
 $EndComp
 $Comp
-L stm8_card-rescue:GND-power #PWR?
+L stm8_card-rescue:GND-power #PWR011
 U 1 1 60B05981
 P 1200 7450
-F 0 "#PWR?" H 1200 7200 50  0001 C CNN
+F 0 "#PWR011" H 1200 7200 50  0001 C CNN
 F 1 "GND" H 1205 7277 50  0000 C CNN
 F 2 "" H 1200 7450 50  0001 C CNN
@@
 3v3
 $Comp
-L stm8_card-rescue:C_Small-Device C?
+L stm8_card-rescue:C_Small-Device C11
 U 1 1 60B15FE3
 P 2450 6650
-F 0 "C?" H 2500 6750 50  0000 L CNN
+F 0 "C11" H 2500 6750 50  0000 L CNN
 F 1 "1uf" H 2500 6550 50  0000 L CNN
 F 2 "Capacitor_SMD:C_0805_2012Metric_Pad1.18x1.45mm_HandSolder" H 2450 6650 50  0001 C CNN
@@
 	2450 6550 2300 6550
 $Comp
-L stm8_card-rescue:GND-power #PWR?
+L stm8_card-rescue:GND-power #PWR012
 U 1 1 60B17629
 P 2450 6750
-F 0 "#PWR?" H 2450 6500 50  0001 C CNN
+F 0 "#PWR012" H 2450 6500 50  0001 C CNN
 F 1 "GND" H 2455 6577 50  0000 C CNN
 F 2 "" H 2450 6750 50  0001 C CNN
@@
 	3200 6450 3750 6450
 $Comp
-L stm8_card-rescue:C_Small-Device C?
+L stm8_card-rescue:C_Small-Device C13
 U 1 1 60B17AD2
 P 3750 6550
-F 0 "C?" H 3700 6750 50  0000 L CNN
+F 0 "C13" H 3700 6750 50  0000 L CNN
 F 1 "1uf" H 3800 6450 50  0000 L CNN
 F 2 "Capacitor_SMD:C_0805_2012Metric_Pad1.18x1.45mm_HandSolder" H 3750 6550 50  0001 C CNN
@@
 $EndComp
 $Comp
-L stm8_card-rescue:GND-power #PWR?
+L stm8_card-rescue:GND-power #PWR015
 U 1 1 60B17FDD
 P 3750 6650
-F 0 "#PWR?" H 3750 6400 50  0001 C CNN
+F 0 "#PWR015" H 3750 6400 50  0001 C CNN
 F 1 "GND" H 3755 6477 50  0000 C CNN
 F 2 "" H 3750 6650 50  0001 C CNN
@@
 $EndComp
 $Comp
-L stm8_card-rescue:C_Small-Device C?
+L stm8_card-rescue:C_Small-Device C12
 U 1 1 60B3D918
 P 3350 6650
-F 0 "C?" H 3400 6750 50  0000 L CNN
+F 0 "C12" H 3400 6750 50  0000 L CNN
 F 1 "0.1uF" H 3400 6550 50  0000 L CNN
 F 2 "Capacitor_SMD:C_0805_2012Metric_Pad1.18x1.45mm_HandSolder" H 3350 6650 50  0001 C CNN
@@
 $EndComp
 $Comp
-L stm8_card-rescue:GND-power #PWR?
+L stm8_card-rescue:GND-power #PWR014
 U 1 1 60B3DF14
 P 3350 6750
-F 0 "#PWR?" H 3350 6500 50  0001 C CNN
+F 0 "#PWR014" H 3350 6500 50  0001 C CNN
 F 1 "GND" H 3355 6577 50  0000 C CNN
 F 2 "" H 3350 6750 50  0001 C CNN
@@
 	3350 6550 3200 6550
 $Comp
-L stm8_card-rescue:R-Device R?
+L stm8_card-rescue:R-Device R8
 U 1 1 60B433B2
 P 4350 6450
-F 0 "R?" V 4250 6450 50  0000 C CNN
+F 0 "R8" V 4250 6450 50  0000 C CNN
 F 1 "470" V 4350 6450 50  0000 C CNN
 F 2 "Resistor_SMD:R_0805_2012Metric_Pad1.20x1.40mm_HandSolder" V 4280 6450 50  0001 C CNN
